File: rascsi_2p1/rascsi_2p1.kicad_pcb (KiCad board)
At the start: 2 copper layers, 65 x 56 mm, 92 parts, among them IC1 SN74LS245DW, IC2 SN74LS245DW, IC3 SN74LS245DW, IC4 SN74LS245DW, J1 Raspberry_Pi_2_3, J2 Conn_01x02_Male, J3 Conn_02x25_Odd_Even, J4 I2C Pinout, J5 L717SDB25PA4CH4F, X1 Mac, X2 Dogcow, X3 Mac2, X4 Raspberry Pi, X5 Dogcow2, X6 Mac Trashcan, X7 Pi, X8 Pi

Commit message: Fixed orientation of termpwr diode. Updated to version "2.1a"
Parts:
- removed X8: Pi, SamacSys_Parts:scsi_logo
- D1, D2, D3, D4, D6: value LED_Small -> Green
- R3, R5, R6: value 147 -> 120
- turned D7 to 270 degrees
Connections:
- D7 pad 1: +5V -> Net-(D7-Pad1)
- D7 pad 2: Net-(D7-Pad2) -> +5V
- FUSE1 pad 1: Net-(D7-Pad2) -> Net-(D7-Pad1)
Routing:
- net GND: track 86.9 -> 69.1 mm, vias 15 -> 107
- net Net-(D7-Pad2): track 4.84 -> 0.00 mm
- net Net-(D7-Pad1): track 0.00 -> 4.84 mm
- net PI-ACT: track 68.4 -> 70.3 mm
- net C-D5: track 61.2 -> 62.9 mm
- net +3V3: track 89.4 -> 90.9 mm
- net C-MSG: track 59.0 -> 60.5 mm
- net C-D2: track 74.1 -> 75.5 mm
- net C-D0: track 64.1 -> 65.0 mm
- net C-D7: track 64.9 -> 65.8 mm
- net C-D3: track 63.8 -> 64.6 mm
- net C-C_D: track 62.1 -> 62.7 mm
- net +5V: track 126.6 -> 127.3 mm
- net (no net): vias 0 -> 4
Other:
- board text added: "68kmla Version 2.1a"
- board text removed: "68kmla Version 2.1"
