File: daisy_chain_board/daisy_chain_board.sch (KiCad schematic (older format))
At the start: 9 parts, among them J7 Conn_02x25_Odd_Even, J8 CONFLY DB25, X1 Mac, X2 Dogcow, X3 Mac2, X4 Raspberry Pi, X7 Pi

Commit message: Fix daisychain board files (#462)
* Revert "Added STEP file and updated symbol and 3d model references to reference the correct gender of parts. Should be no functional change"

This reverts commit 479cc578b885d9d675a35aab40d5217a447c2dfc.

* Delete rascsi_tester that didn't work

Co-authored-by: Tony Kuker <akuker@gmail.com>
Parts:
- J7: footprint Connector_PinSocket_2.54mm:PinSocket_2x25_P2.54mm_Vertical -> Connector_PinHeader_2.54mm:PinHeader_2x25_P2.54mm_Vertical
- J8: footprint SamacSys_Parts:57489011 -> L717SDB25PA4CH4F; symbol SamacSys_Parts:5748901-1 -> SamacSys_Parts:L717SDB25PA4CH4F
Changed lines of the file:
@@
 EESchema Schematic File Version 4
+LIBS:daisy_chain_board-cache
 EELAYER 30 0
 EELAYER END
@@
 F 0 "J7" H 3600 675 50  0000 C CNN
 F 1 "Conn_02x25_Odd_Even" H 3600 766 50  0000 C CNN
-F 2 "Connector_PinSocket_2.54mm:PinSocket_2x25_P2.54mm_Vertical" H 3550 2100 50  0001 C CNN
+F 2 "Connector_PinHeader_2.54mm:PinHeader_2x25_P2.54mm_Vertical" H 3550 2100 50  0001 C CNN
 F 3 "~" H 3550 2100 50  0001 C CNN
 F 4 "C40024" H 3550 2100 50  0001 C CNN "LCSC"
@@
 $EndComp
 $Comp
-L SamacSys_Parts:5748901-1 J8
+L SamacSys_Parts:L717SDB25PA4CH4F J8
 U 1 1 5FA017A4
 P 2900 2900
 F 0 "J8" V 2719 2900 50  0000 C CNN
 F 1 "CONFLY DB25" V 2810 2900 50  0000 C CNN
-F 2 "SamacSys_Parts:57489011" H 4550 3200 50  0001 L CNN
+F 2 "L717SDB25PA4CH4F" H 4550 3200 50  0001 L CNN
 F 3 "https://componentsearchengine.com/Datasheets/1/L717SDB25PA4CH4F.pdf" H 4550 3100 50  0001 L CNN
 F 4 "D-Sub Standard Connectors 25P Size B Stamped Male DSub Contact SD" H 4550 3000 50  0001 L CNN "Description"
@@
 F 10 "C77838" V 2900 2900 50  0001 C CNN "LCSC"
 	1    2900 2900
-	0    1    1    0
+	0    -1   1    0
 $EndComp
 Text Notes 6750 7760 0    87   ~ 17

Commit message: Added STEP file and updated symbol and 3d model references to reference the correct gender of parts. Should be no functional change
Parts:
- J7: footprint Connector_PinHeader_2.54mm:PinHeader_2x25_P2.54mm_Vertical -> Connector_PinSocket_2.54mm:PinSocket_2x25_P2.54mm_Vertical
- J8: footprint L717SDB25PA4CH4F -> SamacSys_Parts:57489011; symbol SamacSys_Parts:L717SDB25PA4CH4F -> SamacSys_Parts:5748901-1
Changed lines of the file:
@@
 EESchema Schematic File Version 4
-LIBS:daisy_chain_board-cache
 EELAYER 30 0
 EELAYER END
@@
 F 0 "J7" H 3600 675 50  0000 C CNN
 F 1 "Conn_02x25_Odd_Even" H 3600 766 50  0000 C CNN
-F 2 "Connector_PinHeader_2.54mm:PinHeader_2x25_P2.54mm_Vertical" H 3550 2100 50  0001 C CNN
+F 2 "Connector_PinSocket_2.54mm:PinSocket_2x25_P2.54mm_Vertical" H 3550 2100 50  0001 C CNN
 F 3 "~" H 3550 2100 50  0001 C CNN
 F 4 "C40024" H 3550 2100 50  0001 C CNN "LCSC"
@@
 $EndComp
 $Comp
-L SamacSys_Parts:L717SDB25PA4CH4F J8
+L SamacSys_Parts:5748901-1 J8
 U 1 1 5FA017A4
 P 2900 2900
 F 0 "J8" V 2719 2900 50  0000 C CNN
 F 1 "CONFLY DB25" V 2810 2900 50  0000 C CNN
-F 2 "L717SDB25PA4CH4F" H 4550 3200 50  0001 L CNN
+F 2 "SamacSys_Parts:57489011" H 4550 3200 50  0001 L CNN
 F 3 "https://componentsearchengine.com/Datasheets/1/L717SDB25PA4CH4F.pdf" H 4550 3100 50  0001 L CNN
 F 4 "D-Sub Standard Connectors 25P Size B Stamped Male DSub Contact SD" H 4550 3000 50  0001 L CNN "Description"
@@
 F 10 "C77838" V 2900 2900 50  0001 C CNN "LCSC"
 	1    2900 2900
-	0    -1   1    0
+	0    1    1    0
 $EndComp
 Text Notes 6750 7760 0    87   ~ 17
