File: rascsi_2p6/Connectors.kicad_sch (KiCad schematic)
At the start: 3 parts, among them J20 171826-4, J3 Conn_02x25_Odd_Even, J9 Conn_02x25_Odd_Even

Commit message: Revert back to original version of rascsi 2.6 board.
This reverts commit 2b424468fa236e169660193e1614c490b0ff0ed6.
Parts:
- J9: now in the parts list
Changed lines of the file:
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@@
   )
   (symbol (lib_id "Connector_Generic:Conn_02x25_Odd_Even") (at 76.2 83.82 270) (unit 1)
-    (in_bom no) (on_board no)
+    (in_bom yes) (on_board yes)
     (property "Reference" "J9" (id 0) (at 40.005 85.09 0))
     (property "Value" "Conn_02x25_Odd_Even" (id 1) (at 42.3164 85.09 0))

Commit message: update silkscreen to say piscsi and regenerate prod files
Parts:
- J9: now left out of the parts list
Changed lines of the file:
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@@
   )
   (symbol (lib_id "Connector_Generic:Conn_02x25_Odd_Even") (at 76.2 83.82 270) (unit 1)
-    (in_bom yes) (on_board yes)
+    (in_bom no) (on_board no)
     (property "Reference" "J9" (id 0) (at 40.005 85.09 0))
     (property "Value" "Conn_02x25_Odd_Even" (id 1) (at 42.3164 85.09 0))
