File: piscsi_2p6/piscsi.kicad_pcb (KiCad board)
At the start: 2 copper layers, 65 x 56 mm, 97 parts, among them IC1 SN74LS641-1DW, IC2 SN74LS641-1DW, IC3 SN74LS641-1DW, IC4 SN74LS641-1DW, J1 Raspberry_Pi_2_3, J2 DNP, J20 171826-4, J3 Conn_02x25_Odd_Even, J4 I2C Pinout, J5 DNP, J6 CONNFLY DB-25, J8 USB_B_Micro, J9 Conn_02x25_Odd_Even, X1 Mac, X2 Dogcow, X3 Mac, X4 Dogcow, X5 Dogcow, X6 Dogcow, X7 Pi, X8 Pi

Commit message: updates
Parts:
- J6: footprint SamacSys_Parts:L717SDB25PA4CH4F -> SamacSys_Parts:L717SDB25PA4CH4F_Flipped; moved to F.Cu
- S1: footprint rascsi_din:SOIC127P812X230-4N -> SamacSys_Parts:SOIC127P812X230-4N
- moved J6 33.2 mm to (190.4, 87.6), turned to 0 degrees
