File: piscsi_2p6/piscsi.kicad_sch (KiCad schematic)
At the start: 88 parts, among them IC1 SN74LS641-1DW, IC2 SN74LS641-1DW, IC3 SN74LS641-1DW, IC4 SN74LS641-1DW, J1 Raspberry_Pi_2_3, J2 DNP, J4 I2C Pinout, J5 DNP, J6 CONNFLY DB-25, X1 Mac, X2 Dogcow, X3 Mac, X4 Dogcow, X5 Dogcow, X6 Dogcow, X7 Pi, X8 Pi

Commit message: updates
Parts:
- J6: footprint L717SDB25PA4CH4F -> SamacSys_Parts:L717SDB25PA4CH4F_Flipped
- S1: footprint rascsi_din:SOIC127P812X230-4N -> SamacSys_Parts:SOIC127P812X230-4N
Changed lines of the file:
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@@
     (property "Reference" "S1" (id 0) (at 92.71 17.78 0))
     (property "Value" "Switch x2" (id 1) (at 107.95 17.78 0))
-    (property "Footprint" "rascsi_din:SOIC127P812X230-4N" (id 2) (at 113.03 19.05 0)
+    (property "Footprint" "SamacSys_Parts:SOIC127P812X230-4N" (id 2) (at 113.03 19.05 0)
       (effects (font (size 1.27 1.27)) (justify left) hide)
     )
@@
     (property "Reference" "J6" (id 0) (at 233.68 67.7926 90))
     (property "Value" "CONNFLY DB-25" (id 1) (at 233.68 70.104 90))
-    (property "Footprint" "L717SDB25PA4CH4F" (id 2) (at 226.06 114.3 0)
+    (property "Footprint" "SamacSys_Parts:L717SDB25PA4CH4F_Flipped" (id 2) (at 226.06 114.3 0)
       (effects (font (size 1.27 1.27)) (justify left) hide)
     )
@@
     )
     (path "/00000000-0000-0000-0000-00005fa017a4"
-      (reference "J6") (unit 1) (value "CONNFLY DB-25") (footprint "L717SDB25PA4CH4F")
+      (reference "J6") (unit 1) (value "CONNFLY DB-25") (footprint "SamacSys_Parts:L717SDB25PA4CH4F_Flipped")
     )
     (path "/00000000-0000-0000-0000-00005fec586e/00000000-0000-0000-0000-00005fec9a88"
@@
     )
     (path "/00000000-0000-0000-0000-00005f38ecd6"
-      (reference "S1") (unit 1) (value "Switch x2") (footprint "rascsi_din:SOIC127P812X230-4N")
+      (reference "S1") (unit 1) (value "Switch x2") (footprint "SamacSys_Parts:SOIC127P812X230-4N")
     )
     (path "/00000000-0000-0000-0000-00005fec586e/00000000-0000-0000-0000-00005fed04f9"
