File: piscsi_2p7/piscsi.kicad_pcb (KiCad board)
At the start: 2 copper layers, 65 x 56 mm, 97 parts, among them IC1 SN74LS641-1DW, IC2 SN74LS641-1DW, IC3 SN74LS641-1DW, IC4 SN74LS641-1DW, J1 Raspberry_Pi_2_3, J2 DNP, J20 171826-4, J3 Conn_02x25_Odd_Even, J4 I2C Pinout, J5 DNP, J6 CONNFLY DB-25, J8 USB_B_Micro, J9 Conn_02x25_Odd_Even, X1 Mac, X2 Dogcow, X3 Mac, X4 Dogcow, X5 Dogcow, X6 Dogcow, X7 Pi, X8 Pi

Commit message: as ordered 2.7
Parts:
- added C1: 10uF, Capacitor_SMD:C_0402_1005Metric, F.Cu at (181.8, 50.6)
- added C2: 10uF, Capacitor_SMD:C_0402_1005Metric, F.Cu at (193.4, 50.6)
- added C3: 10uF, Capacitor_SMD:C_0402_1005Metric, F.Cu at (219.9, 65.5)
- added C4: 10uF, Capacitor_SMD:C_0402_1005Metric, F.Cu at (231.6, 65.8)
- J6: footprint SamacSys_Parts:L717SDB25PA4CH4F -> SamacSys_Parts:L717SDB25PA4CH4F_Flipped; moved to F.Cu
- moved J6 33.2 mm to (190.4, 87.6), turned to 0 degrees
- moved S1 5.45 mm to (207.5, 74.3), turned to 0 degrees
- moved R27 3.25 mm to (210.2, 66.3)
- moved R28 3.25 mm to (212.1, 66.3)
- moved R29 3.25 mm to (214.0, 66.3)
- moved R30 3.25 mm to (215.9, 66.3)
- moved R31 3.25 mm to (217.8, 66.3)
- moved R45 3.25 mm to (210.2, 69.7)
- moved R46 3.25 mm to (212.1, 69.7)
- moved R47 3.25 mm to (214.0, 69.7)
- moved R48 3.25 mm to (215.9, 69.7)
- moved R49 3.25 mm to (217.8, 69.7)
Connections:
- IC1 pad 20: +5V -> +3V3
- IC2 pad 20: +5V -> +3V3
- IC3 pad 20: +5V -> +3V3
- IC4 pad 20: +5V -> +3V3
Routing:
- net +5V: track 244.3 -> 208.4 mm
- net GND: track 484.2 -> 504.6 mm, vias 42 -> 43
- net +3V3: track 147.3 -> 163.6 mm
- net /TERM_GND: track 67.6 -> 70.5 mm
- net C-BSY: track 59.3 -> 62.1 mm
- net C-REQ: track 100.3 -> 98.9 mm
- net C-I_O: track 111.3 -> 110.8 mm
Other:
- board text added: "Version 2.7"
- board text added: "https://github.com/piscsi Copyright 2023 akuker"
- board text removed: "Version 2.6e"
- board text removed: "https://github.com/piscsi Copyright 2022 akuker"
