File: daisy_chain_board_v2/daisy_chain_board.kicad_pcb (KiCad board)
At the start: 2 copper layers, 65 x 21.2 mm, 8 parts, among them J7 Conn_02x25_Odd_Even, J8 CONFLY DB25, X1 Mac, X3 Mac2, X4 Raspberry Pi, X7 Pi

Commit message: rebranded to piscsi
Parts:
- moved X3 0.67 mm to (178.3, 88.2)
Other:
- board text added: "BAD WOLF"
- board text added: "Copyright 2022 akuker"
- board text added: "PiSCSI"
- board text added: "https://github.com/piscsi/piscsi-hw"
- board text removed: "RaSCSI"
- board text removed: "Reloaded"
- board text removed: "https://github.com/akuker/RASCSI"
Changed lines of the file:
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@@
   )
   (footprint "SamacSys_Parts:mac_happy_small" (layer "B.Cu")
-    (at 177.673 88.265 180)
+    (at 178.345364 88.246909 180)
     (property "Sheetfile" "daisy_chain_board.kicad_sch")
     (property "Sheetname" "")
@@
   (gr_line (start 174.5 80.798) (end 174.5 94.996) (layer "Edge.Cuts") (width 0.05))
   (gr_line (start 239.5 80.798) (end 239.5 94.996) (layer "Edge.Cuts") (width 0.05))
-  (gr_text "Reloaded" (at 186.727 96.648) (layer "F.Cu")
-    (effects (font (size 1 1) (thickness 0.15) italic))
-  )
-  (gr_text "RaSCSI" (at 186.727 94.743) (layer "F.Cu")
+  (gr_text "PiSCSI" (at 186.72 95.37) (layer "F.Cu")
     (effects (font (size 2 2) (thickness 0.4) italic))
   )
-  (gr_text "Reloaded" (at 227.273 96.648) (layer "B.Cu")
-    (effects (font (size 1 1) (thickness 0.15) italic) (justify mirror))
-  )
-  (gr_text "RaSCSI" (at 227.273 94.743) (layer "B.Cu")
+  (gr_text "BAD WOLF" (at 175.62 91.69 90) (layer "B.Cu")
+    (effects (font (size 1 1) (thickness 0.15)) (justify mirror))
+  )
+  (gr_text "PiSCSI" (at 227.04 95.42) (layer "B.Cu")
     (effects (font (size 2 2) (thickness 0.4) italic) (justify mirror))
   )
-  (gr_text "https://github.com/akuker/RASCSI" (at 207 97) (layer "B.SilkS")
+  (gr_text "https://github.com/piscsi/piscsi-hw" (at 207 97) (layer "B.SilkS")
     (effects (font (size 1 1) (thickness 0.15)) (justify mirror))
   )
@@
     (effects (font (size 1 0.8) (thickness 0.15)) (justify mirror))
   )
+  (gr_text "Copyright\n2022\nakuker" (at 185.71 94.29) (layer "B.SilkS")
+    (effects (font (size 1 1) (thickness 0.15)) (justify mirror))
+  )
   (gr_text "SCSI Daisy Chain Board" (at 207 94.8) (layer "B.SilkS")
     (effects (font (size 1.5 1.5) (thickness 0.2)) (justify mirror))
   )
-  (gr_text "https://github.com/akuker/RASCSI" (at 207 95.7) (layer "F.SilkS")
+  (gr_text "https://github.com/piscsi/piscsi-hw" (at 207 95.7) (layer "F.SilkS")
     (effects (font (size 1 1) (thickness 0.15)))
   )
@@
     (members
       2ab16679-030c-4500-9313-4ba67d431f36
-      31777d83-d4ac-4bbc-91f5-f3b29a1b2f46
       88d4abda-6003-471e-b0b2-3b6a3a400a1d
       9df3d29b-3af9-4a1b-9695-6d1352a33e27
