File: daisy_chain_board_v2/daisy_chain_board.kicad_sch (KiCad schematic)
At the start: 8 parts, among them J7 Conn_02x25_Odd_Even, J8 CONFLY DB25, X1 Mac, X3 Mac2, X4 Raspberry Pi, X7 Pi

Commit message: rebranded to piscsi
Other:
- note added: "PiSCSI Daisy Chain Board"
- note removed: "RaSCSI Daisy Chain Board"
Changed lines of the file:
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@@
     (effects (font (size 1.4986 1.4986) (thickness 0.2997) bold) (justify left bottom))
   )
-  (text "RaSCSI Daisy Chain Board" (at 171.45 197.104 0)
+  (text "PiSCSI Daisy Chain Board" (at 171.45 197.104 0)
     (effects (font (size 2.2098 2.2098) (thickness 0.442) bold) (justify left bottom))
   )
